File: KiCAD/imu-adapter/imu-adapter.kicad_sch (KiCad schematic)
At the start: 6 parts, among them J1 2x3_0.1in, J2 1mm_SIP

Commit message: Update KiCAD, start software
Parts:
- J1: CatNo (none) -> 2057-PH2-06-UA-ND; MfgNo (none) -> PH2-06-UA
- J2: CatNo (none) -> 2073-BC020-06-A-0200-0300-L-D-ND; MfgNo (none) -> BC020-06-A-0200-0300-L-D
Changed lines of the file:
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@@
+      (effects (font (size 1.27 1.27)) hide)
+    )
+    (property "CatNo" "" (at 40.64 38.1 0)
+      (effects (font (size 1.27 1.27)) hide)
+    )
+    (property "MfgNo" "" (at 40.64 38.1 0)
       (effects (font (size 1.27 1.27)) hide)
     )
@@
       (effects (font (size 1.27 1.27)) hide)
     )
+    (property "CatNo" "" (at 40.64 50.8 0)
+      (effects (font (size 1.27 1.27)) hide)
+    )
+    (property "MfgNo" "" (at 40.64 50.8 0)
+      (effects (font (size 1.27 1.27)) hide)
+    )
     (instances
       (project "imu-adapter"
@@
   )
   (symbol (lib_id "Connector:AVR-ISP-6") (at 83.82 91.44 0) (mirror y) (unit 1)
-    (in_bom yes) (on_board yes) (dnp no) (fields_autoplaced)
+    (in_bom yes) (on_board yes) (dnp no)
     (property "Reference" "J1" (at 92.71 88.9 0)
       (effects (font (size 1.27 1.27)) (justify right))
@@
     )
     (property "Datasheet" " ~" (at 116.205 105.41 0)
+      (effects (font (size 1.27 1.27)) hide)
+    )
+    (property "CatNo" "2057-PH2-06-UA-ND" (at 88.9 105.41 0)
+      (effects (font (size 1.27 1.27)))
+    )
+    (property "MfgNo" "PH2-06-UA" (at 83.82 91.44 0)
       (effects (font (size 1.27 1.27)) hide)
     )
@@
       (effects (font (size 1.27 1.27)) hide)
     )
+    (property "CatNo" "" (at 40.64 44.45 0)
+      (effects (font (size 1.27 1.27)) hide)
+    )
+    (property "MfgNo" "" (at 40.64 44.45 0)
+      (effects (font (size 1.27 1.27)) hide)
+    )
     (instances
       (project "imu-adapter"
@@
     )
     (property "Datasheet" "~" (at 40.64 31.75 0)
+      (effects (font (size 1.27 1.27)) hide)
+    )
+    (property "CatNo" "" (at 40.64 31.75 0)
+      (effects (font (size 1.27 1.27)) hide)
+    )
+    (property "MfgNo" "" (at 40.64 31.75 0)
       (effects (font (size 1.27 1.27)) hide)
     )
@@
       (effects (font (size 1.27 1.27)) hide)
     )
+    (property "CatNo" "2073-BC020-06-A-0200-0300-L-D-ND" (at 50.8 105.41 0)
+      (effects (font (size 1.27 1.27)))
+    )
+    (property "MfgNo" "BC020-06-A-0200-0300-L-D" (at 50.8 91.44 0)
+      (effects (font (size 1.27 1.27)) hide)
+    )
