File: KiCAD/imu-splitter/imu-splitter.kicad_sch (KiCad schematic)
At the start: 18 parts, among them J1 4P4C, J2 4P4C, J3 4P4C, J4 4P4C, J5 4P4C, J6 4P4C, J7 3220-26-0200-00, J8 Conn_01x04, J9 Conn_01x05, U1 AP2114H-3.3TRG1

Commit message: As built V2.0
Parts:
- added J10: 3221-26-0100-00, models:SAMTEC_SHF-113-01-L-D-RA, symbol Connector_Generic:Conn_02x13_Odd_Even
- N1: CatNo (none) -> 164-1551TGY-ND; MfgNo (none) -> 1551TGY
Changed lines of the file:
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@@
+	)
+	(symbol
+		(lib_id "Connector_Generic:Conn_02x13_Odd_Even")
+		(at 88.9 93.98 0)
+		(unit 1)
+		(exclude_from_sim no)
+		(in_bom yes)
+		(on_board no)
+		(dnp yes)
+		(property "Reference" "J10"
+			(at 81.28 72.39 0)
+			(effects
+				(font
+					(size 1.27 1.27)
+				)
+			)
+		)
+		(property "Value" "3221-26-0100-00"
+			(at 99.06 72.39 0)
+			(effects
+				(font
+					(size 1.27 1.27)
+				)
+			)
+		)
+		(property "Footprint" "models:SAMTEC_SHF-113-01-L-D-RA"
+			(at 88.9 93.98 0)
+			(effects
+				(font
+					(size 1.27 1.27)
+				)
+				(hide yes)
+			)
+		)
+		(property "Datasheet" "~"
+			(at 88.9 93.98 0)
+			(effects
+				(font
+					(size 1.27 1.27)
+				)
+				(hide yes)
+			)
+		)
+		(property "Description" ""
+			(at 88.9 93.98 0)
+			(effects
+				(font
+					(size 1.27 1.27)
+				)
+				(hide yes)
+			)
+		)
+		(property "CatNo" "1175-1745-ND"
+			(at 95.25 74.93 0)
+			(effects
+				(font
+					(size 1.27 1.27)
+				)
+			)
+		)
+		(property "MfgNo" "3221-26-0100-00"
+			(at 88.9 93.98 0)
+			(effects
+				(font
+					(size 1.27 1.27)
+				)
+				(hide yes)
+			)
+		)
+		(pin "5"
+		)
+		(pin "8"
+		)
+		(pin "6"
+		)
+		(pin "4"
+		)
+		(pin "13"
+		)
+		(pin "19"
+		)
+		(pin "7"
+		)
+		(pin "25"
+		)
+		(pin "10"
+		)
+		(pin "3"
+		)
+		(pin "2"
+		)
+		(pin "9"
+		)
+		(pin "23"
+		)
+		(pin "26"
+		)
+		(pin "20"
+		)
+		(pin "18"
+		)
+		(pin "24"
+		)
+		(pin "11"
+		)
+		(pin "12"
+		)
+		(pin "21"
+		)
+		(pin "22"
+		)
+		(pin "16"
+		)
+		(pin "15"
+		)
+		(pin "14"
+		)
+		(pin "17"
+		)
+		(pin "1"
+		)
+		(instances
+			(project "imu-splitter"
+				(path "/3ddff065-8308-49ba-816e-3ac23a1c142d"
+					(reference "J10")
+					(unit 1)
+				)
+			)
+		)
 	)
 	(symbol
@@
 		(exclude_from_sim yes)
 		(in_bom yes)
-		(on_board no)
+		(on_board yes)
 		(dnp no)
 		(fields_autoplaced yes)
@@
 			(at 45.72 175.26 0)
 			(effects
+				(font
+					(size 1.27 1.27)
+				)
+				(hide yes)
+			)
+		)
+		(property "CatNo" "164-1551TGY-ND"
+			(at 45.72 175.26 0)
+			(effects
+				(font
+					(size 1.27 1.27)
+				)
+				(hide yes)
+			)
+		)
+		(property "MfgNo" "1551TGY"
+			(at 45.72 175.26 0)
+			(effects
