File: KiCAD/imu-board/imu-board.kicad_pcb (KiCad board)
At the start: 4 copper layers, 11.2 x 17.8 mm, 10 parts, among them J2 A-2004-3-4-LP-N-R, J3 -OMIT-, U2 ISM330DHCX, U3 ATmega168A-MM

Commit message: routing
Parts:
- moved R1 8.21 mm to (52.7, 68.1)
- moved D1 8.21 mm to (52.7, 69.5)
- moved JP1 7.81 mm to (54.6, 54.9), turned to 180 degrees
- moved JP2 7.11 mm to (54.6, 53.7), turned to 180 degrees
- moved C2 1.70 mm to (51.2, 60.2), turned to 90 degrees
- moved U3 0.67 mm to (54.7, 60.2)
Routing:
- net /TXD: track 0.00 -> 18.9 mm, vias 0 -> 2
- net /RXD: track 0.00 -> 13.5 mm, vias 0 -> 2
- net /MISO: track 0.00 -> 9.53 mm
- net /MOSI: track 0.00 -> 9.52 mm, vias 0 -> 1
- net /nRESET: track 0.00 -> 6.83 mm, vias 0 -> 1
- net /SCK: track 0.00 -> 6.35 mm
- net /SCL: track 0.00 -> 3.58 mm
- net VCC: track 2.94 -> 6.50 mm, vias 4 -> 6
- net /SDA: track 0.00 -> 3.15 mm
- net GND: track 8.45 -> 10.7 mm, vias 5 -> 8
- net Net-(D1-A): track 0.00 -> 1.41 mm
Other:
- board size 11.2 x 17.8 mm -> 11.2 x 18 mm

Commit message: revised V2 draft layout for review
Parts:
- moved JP1 16.7 mm to (60.2, 70.6)
- moved JP2 16.0 mm to (60.2, 68.7)
- renumbered U3 to U1
Connections:
- U1 pad 1: Net-(JP2-A) -> unconnected-(U1-PD3-Pad1)
- U1 pad 2: Net-(JP1-A) -> unconnected-(U1-PD4-Pad2)
- U1 pad 20: unconnected-(U3-PC1-Pad20) -> Net-(JP1-A)
- U1 pad 21: unconnected-(U3-PC2-Pad21) -> Net-(JP2-A)
Routing:
- net Net-(U1-PC3): track 0.00 -> 18.3 mm, vias 0 -> 2
- net Net-(JP1-A): track 0.00 -> 10.9 mm, vias 0 -> 2
- net Net-(JP2-A): track 0.00 -> 9.30 mm, vias 0 -> 2
- net /nRESET: track 6.83 -> 8.83 mm
- net GND: track 10.7 -> 11.4 mm
Other:
- board text added: "NN IMU"
- board text added: "V2.0 1/25"
- board text removed: "NN IMU V2.0 1/25"

Commit message: correct gerbers now V2.1
Other:
- board text added: "V2.1 2/25"
- board text removed: "V2.0 1/25"
Changed lines of the file:
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@@
 		(tags "Through hole pin header THT 1x06 1.00mm single row")
 		(property "Reference" "J3"
-			(at 0 -1.56 0)
-			(layer "F.SilkS")
-			(hide yes)
+			(at 1.778 1.714 0)
+			(layer "F.SilkS")
 			(effects
 				(font
@@
 		(layer "Edge.Cuts")
 	)
-	(gr_text "V2.0\n1/25"
+	(gr_text "V2.1\n2/25"
 		(at 61.468 74.93 90)
 		(layer "F.SilkS")

Commit message: as built IMU V2.1
Parts:
- renumbered U1 to U3
Changed lines of the file:
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@@
 	(net 16 "/SCL")
 	(net 17 "/SDA")
-	(net 18 "Net-(U1-PC3)")
-	(net 19 "unconnected-(U1-PD5-Pad7)")
-	(net 20 "unconnected-(U1-XTAL1{slash}PB6-Pad5)")
-	(net 21 "unconnected-(U1-PB1-Pad11)")
-	(net 22 "unconnected-(U1-PB2-Pad12)")
-	(net 23 "unconnected-(U1-XTAL2{slash}PB7-Pad6)")
-	(net 24 "unconnected-(U1-PD4-Pad2)")
-	(net 25 "unconnected-(U1-PD6-Pad8)")
-	(net 26 "unconnected-(U1-PB0-Pad10)")
-	(net 27 "unconnected-(U1-PD3-Pad1)")
-	(net 28 "unconnected-(U1-AREF-Pad17)")
-	(net 29 "unconnected-(U1-PC0-Pad19)")
-	(net 30 "unconnected-(U1-PD2-Pad28)")
-	(net 31 "unconnected-(U1-PD7-Pad9)")
+	(net 18 "Net-(U3-PC3)")
+	(net 19 "unconnected-(U3-PD5-Pad7)")
+	(net 20 "unconnected-(U3-XTAL1{slash}PB6-Pad5)")
+	(net 21 "unconnected-(U3-PB1-Pad11)")
+	(net 22 "unconnected-(U3-PB2-Pad12)")
+	(net 23 "unconnected-(U3-XTAL2{slash}PB7-Pad6)")
+	(net 24 "unconnected-(U3-PD4-Pad2)")
+	(net 25 "unconnected-(U3-PD6-Pad8)")
+	(net 26 "unconnected-(U3-PB0-Pad10)")
+	(net 27 "unconnected-(U3-PD3-Pad1)")
+	(net 28 "unconnected-(U3-AREF-Pad17)")
+	(net 29 "unconnected-(U3-PC0-Pad19)")
+	(net 30 "unconnected-(U3-PD2-Pad28)")
+	(net 31 "unconnected-(U3-PD7-Pad9)")
 	(footprint "Capacitor_SMD:C_0402_1005Metric"
 		(layer "F.Cu")
@@
 		(descr "QFN, 28 Pin (http://ww1.microchip.com/downloads/en/DeviceDoc/8008S.pdf#page=16), generated with kicad-footprint-generator ipc_noLead_generator.py")
 		(tags "QFN NoLead")
-		(property "Reference" "U1"
+		(property "Reference" "U3"
 			(at -2.114 3.095 180)
 			(layer "F.SilkS")
@@
 			(size 0.179289 0.179289)
 			(layers "F.Cu" "F.Paste" "F.Mask")
-			(net 27 "unconnected-(U1-PD3-Pad1)")
+			(net 27 "unconnected-(U3-PD3-Pad1)")
 			(pinfunction "PD3")
 			(pintype "bidirectional")
@@
 			(layers "F.Cu" "F.Paste" "F.Mask")
 			(roundrect_rratio 0.25)
-			(net 24 "unconnected-(U1-PD4-Pad2)")
+			(net 24 "unconnected-(U3-PD4-Pad2)")
 			(pinfunction "PD4")
 			(pintype "bidirectional")
@@
 			(layers "F.Cu" "F.Paste" "F.Mask")
 			(roundrect_rratio 0.25)
-			(net 20 "unconnected-(U1-XTAL1{slash}PB6-Pad5)")
+			(net 20 "unconnected-(U3-XTAL1{slash}PB6-Pad5)")
 			(pinfunction "XTAL1/PB6")
 			(pintype "bidirectional")
@@
 			(layers "F.Cu" "F.Paste" "F.Mask")
 			(roundrect_rratio 0.25)
-			(net 23 "unconnected-(U1-XTAL2{slash}PB7-Pad6)")
+			(net 23 "unconnected-(U3-XTAL2{slash}PB7-Pad6)")
 			(pinfunction "XTAL2/PB7")
 			(pintype "bidirectional")
@@
 			(size 0.179289 0.179289)
 			(layers "F.Cu" "F.Paste" "F.Mask")
-			(net 19 "unconnected-(U1-PD5-Pad7)")
+			(net 19 "unconnected-(U3-PD5-Pad7)")
 			(pinfunction "PD5")
 			(pintype "bidirectional")
@@
 			(size 0.179289 0.179289)
 			(layers "F.Cu" "F.Paste" "F.Mask")
-			(net 25 "unconnected-(U1-PD6-Pad8)")
+			(net 25 "unconnected-(U3-PD6-Pad8)")
 			(pinfunction "PD6")
 			(pintype "bidirectional")
@@
 			(layers "F.Cu" "F.Paste" "F.Mask")
 			(roundrect_rratio 0.25)
-			(net 31 "unconnected-(U1-PD7-Pad9)")
+			(net 31 "unconnected-(U3-PD7-Pad9)")
 			(pinfunction "PD7")
 			(pintype "bidirectional")
@@
 			(layers "F.Cu" "F.Paste" "F.Mask")
 			(roundrect_rratio 0.25)
-			(net 26 "unconnected-(U1-PB0-Pad10)")
+			(net 26 "unconnected-(U3-PB0-Pad10)")
 			(pinfunction "PB0")
 			(pintype "bidirectional")
@@
 			(layers "F.Cu" "F.Paste" "F.Mask")
 			(roundrect_rratio 0.25)
-			(net 21 "unconnected-(U1-PB1-Pad11)")
+			(net 21 "unconnected-(U3-PB1-Pad11)")
 			(pinfunction "PB1")
 			(pintype "bidirectional")
@@
 			(layers "F.Cu" "F.Paste" "F.Mask")
 			(roundrect_rratio 0.25)
-			(net 22 "unconnected-(U1-PB2-Pad12)")
+			(net 22 "unconnected-(U3-PB2-Pad12)")
 			(pinfunction "PB2")
 			(pintype "bidirectional")
@@
 			(layers "F.Cu" "F.Paste" "F.Mask")
 			(roundrect_rratio 0.25)
-			(net 28 "unconnected-(U1-AREF-Pad17)")
+			(net 28 "unconnected-(U3-AREF-Pad17)")
 			(pinfunction "AREF")
 			(pintype "passive")
@@
 			(layers "F.Cu" "F.Paste" "F.Mask")
 			(roundrect_rratio 0.25)
-			(net 29 "unconnected-(U1-PC0-Pad19)")
+			(net 29 "unconnected-(U3-PC0-Pad19)")
 			(pinfunction "PC0")
 			(pintype "bidirectional")
@@
 			(size 0.179289 0.179289)
 			(layers "F.Cu" "F.Paste" "F.Mask")
-			(net 18 "Net-(U1-PC3)")
+			(net 18 "Net-(U3-PC3)")
 			(pinfunction "PC3")
 			(pintype "bidirectional")
@@
 			(size 0.179289 0.179289)
 			(layers "F.Cu" "F.Paste" "F.Mask")
-			(net 30 "unconnected-(U1-PD2-Pad28)")
+			(net 30 "unconnected-(U3-PD2-Pad28)")
 			(pinfunction "PD2")
 			(pintype "bidirectional")
@@
 			(layers "F.Cu" "F.Paste" "F.Mask")
 			(roundrect_rratio 0.25)
-			(net 18 "Net-(U1-PC3)")
+			(net 18 "Net-(U3-PC3)")
 			(pintype "passive")
 		)
